Commit message: sync that in

File: champ_description/urdf/champ.urdf.xacro (robot description, xacro)
@@ -7,5 +7,5 @@
     <link name="base_link">
         <collision>
-            <origin xyz="0 0 0" rpy="0 0 0" />
+            <origin xyz="0 0 0.2" rpy="0 0 0" />
             <geometry>
                 <mesh filename="${base_mesh_path}" scale="0.001 0.001 0.001" />
@@ -40,4 +40,5 @@
     <xacro:champ_leg leg="rf" />
     <xacro:champ_leg leg="rh" />
+    <xacro:include filename="$(find champ_description)/urdf/simulated_full_sensor_suite.xacro" />
     <gazebo>
         <plugin name="p3d_base_controller" filename="libgazebo_ros_p3d.so">
@@ -47,7 +48,7 @@
             </ros>
             <body_name>base_link</body_name>
-            <update_rate>1</update_rate>
-            <xyz_offset>10 10 10</xyz_offset>
-            <rpy_offset>0.1 0.1 0.1</rpy_offset>
+            <update_rate>20</update_rate>
+            <xyz_offset>0 0 0</xyz_offset>
+            <rpy_offset>0.0 0.0 0.0</rpy_offset>
             <gaussian_noise>0.01</gaussian_noise>
         </plugin>

File: champ_description/urdf/leg.urdf.xacro (robot description, xacro)
@@ -86,6 +86,6 @@
         <gazebo reference="${leg}_lower_leg_link">
             <fdir1>1 0 0</fdir1>
-            <mu1>0.2</mu1>
-            <mu2>0.2</mu2>
+            <mu1>100</mu1>
+            <mu2>100</mu2>
             <minDepth>0.001</minDepth>
             <material>Gazebo/Red</material>

File: champ_description/urdf/properties.urdf.xacro (robot description, xacro)
@@ -22,5 +22,5 @@
     <xacro:property name="lower_leg_z_length" value="0.156" />
     <xacro:property name="base_mesh_path" value="file://$(find champ_description)/meshes/base.stl" />
-    <xacro:property name="base_mass" value="4.0" />
+    <xacro:property name="base_mass" value="2.0" />
     <xacro:property name="base_x_length" value="0.5" />
     <xacro:property name="base_y_length" value="0.29" />
