Commit message: recorrect use_sim_time arg

File: champ_description/urdf/simulated_full_sensor_suite.xacro (robot description, xacro)
@@ -22,5 +22,5 @@
     <parent link="base_link" />
     <child link="base_sensor_link" />
-    <origin xyz="0.0 0 0.1" rpy="0 0 0" />
+    <origin xyz="0.0 0 0.4" rpy="0 0 0" />
   </joint>
   <joint name="imu_joint" type="fixed">
