Commit message: sync

File: champ_description/urdf/properties.urdf.xacro (robot description, xacro)
@@ -22,5 +22,5 @@
     <xacro:property name="lower_leg_z_length" value="0.156" />
     <xacro:property name="base_mesh_path" value="file://$(find champ_description)/meshes/base.stl" />
-    <xacro:property name="base_mass" value="6.0" />
+    <xacro:property name="base_mass" value="4.0" />
     <xacro:property name="base_x_length" value="0.5" />
     <xacro:property name="base_y_length" value="0.29" />
