Commit message: gunna cont tmr

File: champ_description/urdf/leg.urdf.xacro (robot description, xacro)
@@ -85,7 +85,9 @@
         </link>
         <gazebo reference="${leg}_lower_leg_link">
-            <fdir1>1 0 0</fdir1>
-            <mu1>100</mu1>
-            <mu2>100</mu2>
+            <kp>1000000.0</kp>
+            <kd>1.0</kd>
+            <mu1>0.8</mu1>
+            <mu2>0.8</mu2>
+            <maxVel>0.0</maxVel>
             <minDepth>0.001</minDepth>
             <material>Gazebo/Red</material>

File: champ_description/urdf/properties.urdf.xacro (robot description, xacro)
@@ -22,5 +22,5 @@
     <xacro:property name="lower_leg_z_length" value="0.156" />
     <xacro:property name="base_mesh_path" value="file://$(find champ_description)/meshes/base.stl" />
-    <xacro:property name="base_mass" value="2.0" />
+    <xacro:property name="base_mass" value="6.0" />
     <xacro:property name="base_x_length" value="0.5" />
     <xacro:property name="base_y_length" value="0.29" />

Commit message: isolate libchamp for now

File: champ_description/urdf/leg.urdf.xacro (robot description, xacro)
@@ -105,4 +105,5 @@
             <child link="${leg}_hip_link" />
             <origin xyz="${base_to_hip_xyz}" rpy="0 0 0" />
+            <dynamics damping="0.0" friction="1.0" />
         </joint>
         <joint name="${leg}_upper_leg_joint" type="revolute">
@@ -112,4 +113,5 @@
             <child link="${leg}_upper_leg_link" />
             <origin xyz="0 ${hip_to_upper_leg} 0" rpy="0 0 0" />
+            <dynamics damping="0.0" friction="1.0" />
         </joint>
         <joint name="${leg}_lower_leg_joint" type="revolute">
@@ -119,4 +121,5 @@
             <child link="${leg}_lower_leg_link" />
             <origin xyz="0 0 -${upper_leg_to_lower_leg_distance}" rpy="0 0 0" />
+            <dynamics damping="0.0" friction="1.0" />
         </joint>
         <joint name="${leg}_foot_joint" type="fixed">
@@ -158,34 +161,4 @@
             </joint>
         </ros2_control>
-        <transmission name="${leg}_hip_joint_trans">
-            <type>transmission_interface/SimpleTransmission</type>
-            <joint name="${leg}_hip_joint">
-                <hardwareInterface>hardware_interface/EffortJointInterface</hardwareInterface>
-            </joint>
-            <actuator name="${leg}_hip_joint_motor">
-                <hardwareInterface>hardware_interface/EffortJointInterface</hardwareInterface>
-                <mechanicalReduction>1</mechanicalReduction>
-            </actuator>
-        </transmission>
-        <transmission name="${leg}_upper_leg_joint_trans">
-            <type>transmission_interface/SimpleTransmission</type>
-            <joint name="${leg}_upper_leg_joint">
-                <hardwareInterface>hardware_interface/EffortJointInterface</hardwareInterface>
-            </joint>
-            <actuator name="${leg}_upper_leg_joint_motor">
-                <hardwareInterface>hardware_interface/EffortJointInterface</hardwareInterface>
-                <mechanicalReduction>1</mechanicalReduction>
-            </actuator>
-        </transmission>
-        <transmission name="${leg}_lower_leg_joint_trans">
-            <type>transmission_interface/SimpleTransmission</type>
-            <joint name="${leg}_lower_leg_joint">
-                <hardwareInterface>hardware_interface/EffortJointInterface</hardwareInterface>
-            </joint>
-            <actuator name="${leg}_lower_joint_motor">
-                <hardwareInterface>hardware_interface/EffortJointInterface</hardwareInterface>
-                <mechanicalReduction>1</mechanicalReduction>
-            </actuator>
-        </transmission>
     </xacro:macro>
 </robot>

File: champ_description/urdf/properties.urdf.xacro (robot description, xacro)
@@ -22,5 +22,5 @@
     <xacro:property name="lower_leg_z_length" value="0.156" />
     <xacro:property name="base_mesh_path" value="file://$(find champ_description)/meshes/base.stl" />
-    <xacro:property name="base_mass" value="4.0" />
+    <xacro:property name="base_mass" value="2.0" />
     <xacro:property name="base_x_length" value="0.5" />
     <xacro:property name="base_y_length" value="0.29" />

Commit message: ...

File: champ_description/urdf/leg.urdf.xacro (robot description, xacro)
@@ -85,13 +85,20 @@
         </link>
         <gazebo reference="${leg}_lower_leg_link">
-            <kp>1000000.0</kp>
-            <kd>1.0</kd>
-            <mu1>0.8</mu1>
-            <mu2>0.8</mu2>
-            <maxVel>0.0</maxVel>
-            <minDepth>0.001</minDepth>
-            <material>Gazebo/Red</material>
+            <material>Gazebo/FlatBlack</material>
+            <mu1>1.0</mu1>
+            <mu2>1.0</mu2>
+            <minDepth>0.0002</minDepth>
+            <kp value="1000000.0" />
+            <kd value="100.0" />
         </gazebo>
         <link name="${leg}_foot_link" />
+        <gazebo reference="${leg}_foot_link">
+            <material>Gazebo/FlatBlack</material>
+            <mu1>1.0</mu1>
+            <mu2>1.0</mu2>
+            <minDepth>0.0002</minDepth>
+            <kp value="1000000.0" />
+            <kd value="100.0" />
+        </gazebo>
         <joint name="${leg}_debug_joint" type="fixed">
             <parent link="base_link" />
@@ -105,4 +112,5 @@
             <child link="${leg}_hip_link" />
             <origin xyz="${base_to_hip_xyz}" rpy="0 0 0" />
+            <dynamics damping="0.1" friction="1000.0" />
         </joint>
         <joint name="${leg}_upper_leg_joint" type="revolute">
@@ -112,4 +120,5 @@
             <child link="${leg}_upper_leg_link" />
             <origin xyz="0 ${hip_to_upper_leg} 0" rpy="0 0 0" />
+            <dynamics damping="0.1" friction="1000.0" />
         </joint>
         <joint name="${leg}_lower_leg_joint" type="revolute">
@@ -119,4 +128,5 @@
             <child link="${leg}_lower_leg_link" />
             <origin xyz="0 0 -${upper_leg_to_lower_leg_distance}" rpy="0 0 0" />
+            <dynamics damping="0.1" friction="1000.0" />
         </joint>
         <joint name="${leg}_foot_joint" type="fixed">
@@ -125,4 +135,5 @@
             <!-- <origin xyz="0.00325 0 -${lower_leg_to_foot_distance}" rpy="0 0 0" /> -->
             <origin xyz="0 0 -${lower_leg_to_foot_distance}" rpy="0 0 0" />
+            <dynamics damping="0.1" friction="1000.0" />
         </joint>
         <ros2_control name="GazeboSystem" type="system">
@@ -165,5 +176,5 @@
             <actuator name="${leg}_hip_joint_motor">
                 <hardwareInterface>hardware_interface/EffortJointInterface</hardwareInterface>
-                <mechanicalReduction>1</mechanicalReduction>
+                <mechanicalReduction>5</mechanicalReduction>
             </actuator>
         </transmission>
@@ -175,5 +186,5 @@
             <actuator name="${leg}_upper_leg_joint_motor">
                 <hardwareInterface>hardware_interface/EffortJointInterface</hardwareInterface>
-                <mechanicalReduction>1</mechanicalReduction>
+                <mechanicalReduction>5</mechanicalReduction>
             </actuator>
         </transmission>
@@ -185,5 +196,5 @@
             <actuator name="${leg}_lower_joint_motor">
                 <hardwareInterface>hardware_interface/EffortJointInterface</hardwareInterface>
-                <mechanicalReduction>1</mechanicalReduction>
+                <mechanicalReduction>5</mechanicalReduction>
             </actuator>
         </transmission>

Commit message: add the spot

File: champ_description/urdf/leg.urdf.xacro (robot description, xacro)
@@ -86,18 +86,46 @@
         <gazebo reference="${leg}_lower_leg_link">
             <material>Gazebo/FlatBlack</material>
-            <mu1>1.0</mu1>
-            <mu2>1.0</mu2>
-            <minDepth>0.0002</minDepth>
-            <kp value="1000000.0" />
-            <kd value="100.0" />
+            <collision>
+                <surface>
+                    <friction>
+                        <ode>
+                            <mu>100</mu>
+                            <mu2>100</mu2>
+                            <slip1>0</slip1>
+                            <slip2>0</slip2>
+                        </ode>
+                    </friction>
+                    <contact>
+                        <ode>
+                            <kp>1000000.0</kp>
+                            <kd>100.0</kd>
+                            <min_depth>0.001</min_depth>
+                        </ode>
+                    </contact>
+                </surface>
+            </collision>
         </gazebo>
         <link name="${leg}_foot_link" />
         <gazebo reference="${leg}_foot_link">
             <material>Gazebo/FlatBlack</material>
-            <mu1>1.0</mu1>
-            <mu2>1.0</mu2>
-            <minDepth>0.0002</minDepth>
-            <kp value="1000000.0" />
-            <kd value="100.0" />
+            <collision>
+                <surface>
+                    <friction>
+                        <ode>
+                            <mu>100</mu>
+                            <mu2>100</mu2>
+                            <slip1>0</slip1>
+                            <slip2>0</slip2>
+                        </ode>
+                    </friction>
+                    <contact>
+                        <ode>
+                            <kp>1000000.0</kp>
+                            <kd>100.0</kd>
+                            <min_depth>0.001</min_depth>
+                        </ode>
+                    </contact>
+                </surface>
+            </collision>
         </gazebo>
         <joint name="${leg}_debug_joint" type="fixed">
@@ -176,5 +204,5 @@
             <actuator name="${leg}_hip_joint_motor">
                 <hardwareInterface>hardware_interface/EffortJointInterface</hardwareInterface>
-                <mechanicalReduction>5</mechanicalReduction>
+                <mechanicalReduction>1</mechanicalReduction>
             </actuator>
         </transmission>
@@ -186,5 +214,5 @@
             <actuator name="${leg}_upper_leg_joint_motor">
                 <hardwareInterface>hardware_interface/EffortJointInterface</hardwareInterface>
-                <mechanicalReduction>5</mechanicalReduction>
+                <mechanicalReduction>1</mechanicalReduction>
             </actuator>
         </transmission>
@@ -196,5 +224,5 @@
             <actuator name="${leg}_lower_joint_motor">
                 <hardwareInterface>hardware_interface/EffortJointInterface</hardwareInterface>
-                <mechanicalReduction>5</mechanicalReduction>
+                <mechanicalReduction>1</mechanicalReduction>
             </actuator>
         </transmission>
