Commit message: champ should be default for now

File: champ_description/urdf/champ/leg.urdf.xacro (robot description, xacro)
@@ -90,6 +90,6 @@
                     <friction>
                         <ode>
-                            <mu>100</mu>
-                            <mu2>100</mu2>
+                            <mu>1</mu>
+                            <mu2>1</mu2>
                             <slip1>0</slip1>
                             <slip2>0</slip2>
@@ -140,5 +140,5 @@
             <child link="${leg}_hip_link" />
             <origin xyz="${base_to_hip_xyz}" rpy="0 0 0" />
-            <dynamics damping="0.1" friction="1000.0" />
+            <dynamics damping="0.7" friction="100.0" />
         </joint>
         <joint name="${leg}_upper_leg_joint" type="revolute">
@@ -148,5 +148,5 @@
             <child link="${leg}_upper_leg_link" />
             <origin xyz="0 ${hip_to_upper_leg} 0" rpy="0 0 0" />
-            <dynamics damping="0.1" friction="1000.0" />
+            <dynamics damping="0.7" friction="100.0" />
         </joint>
         <joint name="${leg}_lower_leg_joint" type="revolute">
@@ -156,5 +156,5 @@
             <child link="${leg}_lower_leg_link" />
             <origin xyz="0 0 -${upper_leg_to_lower_leg_distance}" rpy="0 0 0" />
-            <dynamics damping="0.1" friction="1000.0" />
+            <dynamics damping="0.7" friction="100.0" />
         </joint>
         <joint name="${leg}_foot_joint" type="fixed">
@@ -163,5 +163,5 @@
             <!-- <origin xyz="0.00325 0 -${lower_leg_to_foot_distance}" rpy="0 0 0" /> -->
             <origin xyz="0 0 -${lower_leg_to_foot_distance}" rpy="0 0 0" />
-            <dynamics damping="0.1" friction="1000.0" />
+            <dynamics damping="0.7" friction="100.0" />
         </joint>
         <ros2_control name="GazeboSystem" type="system">

File: champ_description/urdf/spot/spot_leg.urdf.xacro (robot description, xacro)
@@ -6,10 +6,10 @@
     <xacro:arg name="leg_mu2" default="1.0" />
     <xacro:arg name="leg_fdir1" default="" />
-    <xacro:arg name="max_knee_effort" default="160" />
-    <xacro:arg name="max_knee_velocity" default="30" />
-    <xacro:arg name="max_hip_x_effort" default="160" />
-    <xacro:arg name="max_hip_x_velocity" default="30" />
-    <xacro:arg name="max_hip_y_effort" default="160" />
-    <xacro:arg name="max_hip_y_velocity" default="30" />
+    <xacro:arg name="max_knee_effort" default="80" />
+    <xacro:arg name="max_knee_velocity" default="15" />
+    <xacro:arg name="max_hip_x_effort" default="80" />
+    <xacro:arg name="max_hip_x_velocity" default="15" />
+    <xacro:arg name="max_hip_y_effort" default="80" />
+    <xacro:arg name="max_hip_y_velocity" default="15" />
     <xacro:macro name="spot_leg" params="leg_name prefix">
         <xacro:if value="${leg_name == 'front_left'}">
@@ -51,5 +51,5 @@
             <child link="${prefix}${leg_name}_hip" />
             <limit effort="$(arg max_hip_x_effort)" velocity="$(arg max_hip_x_velocity)" lower="-0.78539816339744827899" upper="0.78539816339744827899" />
-            <dynamics damping="0.0" friction="0.0" />
+            <dynamics damping="10.0" friction="100.0" />
         </joint>
         <link name="${prefix}${leg_name}_upper_leg">
@@ -76,5 +76,5 @@
             <child link="${prefix}${leg_name}_upper_leg" />
             <limit effort="$(arg max_hip_y_effort)" velocity="$(arg max_hip_y_velocity)" lower="-0.89884456477707963539" upper="2.2951079663725435509" />
-            <dynamics damping="0.0" friction="0.0" />
+            <dynamics damping="10.0" friction="100.0" />
         </joint>
         <link name="${prefix}${leg_name}_lower_leg">
@@ -122,5 +122,5 @@
             <child link="${prefix}${leg_name}_lower_leg" />
             <limit effort="$(arg max_knee_effort)" velocity="$(arg max_knee_velocity)" lower="-2.7929" upper="-0.254801" />
-            <dynamics damping="0.0" friction="0.0" />
+            <dynamics damping="10.0" friction="100.0" />
         </joint>
         <xacro:empty_link name="${prefix}${leg_name}_ee" />
